Commit message: feat(demo): blue bicycle body and interactive Nav2 kinematic demo
Replace the demo's custom car-like bicycle with a self-authored blue single-track bicycle (bike.urdf, primitive frame/fork/handlebar/wheels, Apache-2.0); the two demo visual URDFs are named by their source assets (r2d2.urdf, bike.urdf) and the standalone launch maps model to body, while the kinematic Model plugins stay Unicycle/Bicycle.

Add prox_mpc_benchmark/launch/interactive.launch.py: the b2 Nav2 stack (kinematic plant + ProxMPC + costmaps) with RViz and the Nav2 Goal tool, so either model can be driven to clicked goals without Gazebo. It lives in the benchmark package because that owns the kinematic plant and Nav2 base config. Refresh the demo README, RViz profiles, Nav2/standalone configs and worlds, and the doc/ guides.

File: prox_mpc_demo/urdf/bike.urdf (robot description, URDF)
Before this commit: robot bike, 6 links, 5 joints
Links:
- removed link chassis
- removed link rear_left_wheel
- removed link rear_right_wheel
- removed link steering_link
- added link frame; visual box size=0.24 0.08 0.04; visual cylinder length=0.058 radius=0.035
- added link handlebar; visual cylinder length=0.50 radius=0.025
- added link rear_wheel; visual cylinder length=0.05 radius=0.35
- link front_wheel: geometry visual cylinder length=0.05 radius=0.35
Joints:
- removed joint base_to_chassis
- removed joint rear_left_wheel_joint
- removed joint rear_right_wheel_joint
- removed joint steering_joint
- added joint base_to_frame: type fixed, parent base_link, child frame, origin xyz=0 0 0
- added joint handlebar_joint: type fixed, parent frame, child handlebar, origin xyz=0.58 0 1.00
- added joint rear_wheel_joint: type fixed, parent base_link, child rear_wheel, origin xyz=-0.8 0 0.35
- joint front_wheel_joint: origin xyz=0 0 0 -> xyz=0.8 0 0.35; parent steering_link -> base_link

File: prox_mpc_demo/worlds/prox_mpc_open.sdf.xacro (robot description, xacro)
@@ -1,5 +1,5 @@
 <?xml version="1.0"?>
 <!--
-  Open-room ProxMPC world for the clean SUCCEEDED gate.
+  Open-room ProxMPC world for open-space navigation.
   A 6x6 m room (walls at +/-3.0 m, inner face ~2.95 m) with an empty interior, so
   the controller drives to the goal in open space (its smooth-tracking regime,

File: prox_mpc_demo/worlds/prox_mpc_world.sdf.xacro (robot description, xacro)
@@ -12,5 +12,5 @@
   Custom robot models and extra obstacles can also be spawned into the running
   world at runtime with `ros2 run ros_gz_sim create ...` (the UserCommands system
-  below enables runtime insertion). See NAV2_SIMULATION.md.
+  below enables runtime insertion). See doc/nav2-simulation.md.
   Args:
     headless   (default true)  : drop the SceneBroadcaster when headless.
